File: KiCad/Motor_Driver.kicad_sch (KiCad schematic)
At the start: 28 parts, among them J1 Battery Terminal, Q1 NMOS, Q2 NMOS, Q3 NMOS, Q4 NMOS, Q5 NMOS, Q6 NMOS, SW1 DIR+A, SW2 DIR-A, U1 PS2801-4

Commit message: Low Side Driver
Parts:
- removed R_Discharge_Path1: 100k, Resistor_THT:R_Axial_DIN0204_L3.6mm_D1.6mm_P5.08mm_Horizontal, symbol Device:R
- removed R_Gate-Protect_AQ1, R_Gate-Protect_AQ2, R_Gate-Protect_AQ3, R_Gate-Protect_AQ4: 10, Resistor_THT:R_Axial_DIN0204_L3.6mm_D1.6mm_P5.08mm_Horizontal, symbol Device:R
- removed R_ILim1, R_ILim2, R_ILim3, R_ILim4: 390, Resistor_THT:R_Axial_DIN0204_L3.6mm_D1.6mm_P5.08mm_Horizontal, symbol Device:R
- removed R_Pull-Down_AQ1, R_Pull-Down_AQ2, R_Pull-Down_AQ3, R_Pull-Down_AQ4: 22k, Resistor_THT:R_Axial_DIN0204_L3.6mm_D1.6mm_P5.08mm_Horizontal, symbol Device:R
- added 12V-J1, 12V-J2: J-12V, Connector_PinHeader_2.54mm:PinHeader_1x02_P2.54mm_Vertical, symbol Jumper:Jumper_2_Open
- added C1: 10uF, Capacitor_THT:CP_Radial_D5.0mm_P2.50mm, symbol Device:C_Polarized_US
- added C2: 1uF, symbol Device:C
- added C3: 100nF, symbol Device:C
- added D4: 1N4007, Diode_THT:D_DO-41_SOD81_P10.16mm_Horizontal, symbol Diode:1N4007
- added D6: 1N5822, Diode_THT:D_DO-201AD_P15.24mm_Horizontal, symbol Diode:1N5822
- added JP1: 24V-J1, Connector_PinHeader_2.54mm:PinHeader_1x02_P2.54mm_Vertical, symbol Jumper:Jumper_2_Bridged
- added L1: 10mH, Inductor_THT:L_Axial_L5.3mm_D2.2mm_P7.62mm_Horizontal_Vishay_IM-1, symbol Device:L
- added L2: 47mH, Inductor_THT:L_Toroid_Vertical_L22.4mm_W10.2mm_P7.90mm_Vishay_TJ4, symbol Device:L
- added Q7: NMOS, Package_TO_SOT_THT:TO-220-3_Vertical, symbol Tesla_Lib:NMOS
- added R1: 500, Resistor_THT:R_Axial_DIN0204_L3.6mm_D1.6mm_P5.08mm_Horizontal, symbol Device:R_US
- added R2: 10k, Resistor_THT:R_Axial_DIN0204_L3.6mm_D1.6mm_P5.08mm_Horizontal, symbol Device:R_US
- added R3: 270, Resistor_THT:R_Axial_DIN0204_L3.6mm_D1.6mm_P5.08mm_Horizontal, symbol Device:R_US
- added R4: 3.3k, Resistor_THT:R_Axial_DIN0204_L3.6mm_D1.6mm_P5.08mm_Horizontal, symbol Device:R_US
- added R_Discharge_Path1, R_Pull-Down_AQ1, R_Pull-Down_AQ2, R_Pull-Down_AQ3, R_Pull-Down_AQ4: 100k, Resistor_THT:R_Axial_DIN0204_L3.6mm_D1.6mm_P5.08mm_Horizontal, symbol Device:R_US
- added R_Gate-Protect_AQ1, R_Gate-Protect_AQ2, R_Gate-Protect_AQ3, R_Gate-Protect_AQ4: 100, Resistor_THT:R_Axial_DIN0204_L3.6mm_D1.6mm_P5.08mm_Horizontal, symbol Device:R_US
- added R_ILim1, R_ILim2, R_ILim3, R_ILim4: 250, Resistor_THT:R_Axial_DIN0204_L3.6mm_D1.6mm_P5.08mm_Horizontal, symbol Device:R_US
- added U1: XL4015, Package_TO_SOT_SMD:TO-263-5_TabPin3, symbol Regulator_Switching:XL4015
- added U4: LM317T, Package_TO_SOT_THT:TO-220F-3_Vertical, symbol dk_PMIC-Voltage-Regulators-Linear:LM317T
- D1, D2, D3: footprint Diode_THT:D_DO-35_SOD27_P7.62mm_Horizontal -> Diode_THT:D_DO-41_SOD81_P10.16mm_Horizontal
- D5: renamed from D4; footprint Diode_THT:D_DO-35_SOD27_P7.62mm_Horizontal -> Diode_THT:D_DO-41_SOD81_P10.16mm_Horizontal
- F1: footprint (none) -> Fuse:Fuseholder_Cylinder-5x20mm_Schurter_0031_8201_Horizontal_Open
- SW1, SW2: footprint (none) -> Button_Switch_THT:Push_E-Switch_KS01Q01
- renumbered U1 to U2
Connections:
- net RPP_Source is gone; now on net GND: Q5.3 (S), Q6.3 (S)
- net EmtrA1: now also R_Gate-Protect_AQ1.1
- net EmtrA2: now also R_Gate-Protect_AQ4.1
- net EmtrA3: now also R_Gate-Protect_AQ3.1
- net EmtrA4: now also R_Gate-Protect_AQ2.1
- net GND: now also C1.2, C2.2, C3.2, Q7.3 (S), R2.1, R4.1, R_Pull-Down_AQ1.1, R_Pull-Down_AQ2.1, R_Pull-Down_AQ3.1, R_Pull-Down_AQ4.1
- net GPow_Q1A: now also R_Gate-Protect_AQ1.2, R_Pull-Down_AQ1.2
- net GPow_Q2A: now also R_Gate-Protect_AQ4.2, R_Pull-Down_AQ2.2
- net GPow_Q3A: now also R_Gate-Protect_AQ3.2, R_Pull-Down_AQ3.2
- net GPow_Q4A: now also R_Gate-Protect_AQ2.2, R_Pull-Down_AQ4.2
- net GSig_Q1A: now also R_ILim1.1
- net GSig_Q2A: now also R_ILim2.1
- net GSig_Q3A: now also R_ILim3.1
- net GSig_Q4A: now also R_ILim4.1
- net ML-A: now also R_Discharge_Path1.1
- net MR-A: now also R_Discharge_Path1.2
- net V_HS-A: now also 12V-J2.1 (A), C1.1, D4.1 (K), R2.2
- net V_LS-A: now also C2.1, R3.2, U4.2 (OUT)
- net Vcc: now also 12V-J1.1 (A), JP1.1 (A), R1.2
- net at U2.3 (A2): now also R_ILim2.2
- net +5V: now reaches SW2.1
- net +5V: now also SW1.1, SW1.3, SW2.3
- net at U2.5 (A3): now also R_ILim3.2
- net at U2.7 (A4): now also R_ILim4.2
- net at U2.1 (A1): now also R_ILim1.2
- new net: 12V-J1.2 (B), L1.1, R1.1
- new net: D4.2 (A), L1.2, Q7.2 (D)
- new net: 12V-J2.2 (B), C3.1, JP1.2 (B), U4.3 (IN)
- new net: R3.1, R4.2, U4.1 (ADJ)
- new net V_Gate-Boost: Q7.1 (G)
Other:
- note added: "Output filter capacitors indication leds"
- note added: "add 2 resistors"
- note removed: "GVO is a fn of SVI with a offset of Vgs (10v) of the NMOS"
- moved on the sheet: F1, J1, SW1, SW2, U2

Commit message: 5v5A supply
Parts:
- removed SW1: DIR+A, Button_Switch_THT:Push_E-Switch_KS01Q01, symbol Switch:SW_DPST
- removed SW2: DIR-A, Button_Switch_THT:Push_E-Switch_KS01Q01, symbol Switch:SW_DPST
- added 5V-J1, 5V-J2: J-12V, Connector_PinHeader_2.54mm:PinHeader_1x02_P2.54mm_Vertical, symbol Jumper:Jumper_2_Open
- added C4, C6, C7: 1uF, Capacitor_THT:C_Disc_D9.0mm_W5.0mm_P5.00mm, symbol Device:C
- added C5: 220uF, Capacitor_THT:CP_Radial_D5.0mm_P2.50mm, symbol Device:C_Polarized_US
- added C8: 330uF, Capacitor_THT:CP_Radial_D5.0mm_P2.50mm, symbol Device:C_Polarized_US
- added J3: Screw_Terminal_01x05, symbol Connector:Screw_Terminal_01x05
- added J4: Motor_A, Connector_AMASS:AMASS_XT60-F_1x02_P7.20mm_Vertical, symbol Connector:Screw_Terminal_01x02
- added R5: 10k, Resistor_THT:R_Axial_DIN0204_L3.6mm_D1.6mm_P5.08mm_Horizontal, symbol Device:R_US
- added R6: 3.3k, Resistor_THT:R_Axial_DIN0204_L3.6mm_D1.6mm_P5.08mm_Horizontal, symbol Device:R_US
- added SW3: DIR+A, symbol Switch:SW_SPST
- added SW4: DIR-A, symbol Switch:SW_SPST
- C2: renamed from C3; footprint (none) -> Capacitor_THT:C_Disc_D9.0mm_W5.0mm_P5.00mm
- C3: renamed from C2; footprint (none) -> Capacitor_THT:C_Disc_D9.0mm_W5.0mm_P5.00mm
- renumbered D4 to D1, D1 to D2, D2 to D3, D3 to D4, Q7 to Q3, Q3 to Q4, Q4 to Q5, Q5 to Q6, Q6 to Q7, R_Gate-Protect_AQ4 to R_Gate-Protect_AQ2, R_Gate-Protect_AQ2 to R_Gate-Protect_AQ4, U4 to U1, U1 to U3
Connections:
- net GSig_Q3A is gone; now on net GSig_Q2A: R_ILim3.1
- net GSig_Q4A is gone; now on net GSig_Q1A: R_ILim4.1
- net +5V: now also 5V-J1.2 (B), J3.2 (Pin_2), SW3.1 (A), SW4.1 (A)
- net GND: now also 5V-J2.1 (A)
- net GND2: now also D6.2 (A), U3.1 (GND), 5V-J2.2 (B), C5.2, C6.2, C7.2, C8.2, J3.1 (Pin_1), R6.1
- net GSig_Q1A: now also J3.3 (Pin_3), SW3.2 (B)
- net GSig_Q2A: now also J3.4 (Pin_4), SW4.2 (B)
- net ML-A: now also J4.1 (Pin_1)
- net MR-A: now also J4.2 (Pin_2)
- net Vcc: now also U3.5 (VIN), C4.1, C5.1, C6.1
- net at U3.2 (FB): now also R5.1, R6.2
- net at U3.3 (SW): now also D6.1 (K), L2.1
- net at U3.4 (VC): now also C4.2
- net at L2.2: now also 5V-J1.1 (A), C7.1, C8.1, R5.2
Other:
- note added: "!! Idiot Proof the H-Bridge !!"
- note added: "Output filter capacitors indication leds On indication LEDs"
- note removed: "Output filter capacitors indication leds"
- moved on the sheet: D6, F1, J1, L2, R_ILim1, R_ILim2, R_ILim3, R_ILim4, U2, U3

Commit message: Short Circuit Protection
Parts:
- removed J3: Screw_Terminal_01x05, symbol Connector:Screw_Terminal_01x05
- removed R_Discharge_Path1: 100k, Resistor_THT:R_Axial_DIN0204_L3.6mm_D1.6mm_P5.08mm_Horizontal, symbol Device:R_US
- added C10: (no value), Capacitor_THT:C_Disc_D9.0mm_W5.0mm_P5.00mm, symbol Device:C
- added C9: 100nF, Capacitor_THT:C_Disc_D9.0mm_W5.0mm_P5.00mm, symbol Device:C
- added D10, D12, D8: 1N4007, Diode_THT:D_DO-41_SOD81_P10.16mm_Horizontal, symbol Diode:1N4007
- added D11: GREEN, LED_THT:LED_D3.0mm, symbol Device:LED
- added D7, D9: BLUE, LED_THT:LED_D3.0mm_Clear, symbol Device:LED
- added J3: MCU Terminals, Connector_JST:JST_EH_B7B-EH-A_1x07_P2.50mm_Vertical, symbol Connector:Screw_Terminal_01x07
- added Q8: AO3405, Package_TO_SOT_SMD:SOT-23, symbol Transistor_FET:AO3401A
- added Q9: AO3400A, Package_TO_SOT_SMD:SOT-23, symbol Transistor_FET:AO3400A
- added R10: 10k, Resistor_THT:R_Axial_DIN0204_L3.6mm_D1.6mm_P5.08mm_Horizontal, symbol Device:R_US
- added R11, R12: ~, Resistor_THT:R_Axial_DIN0204_L3.6mm_D1.6mm_P5.08mm_Horizontal, symbol Device:R_US
- added R7, R8: 1.2k, Resistor_THT:R_Axial_DIN0204_L3.6mm_D1.6mm_P5.08mm_Horizontal, symbol Device:R_US
- added R9: 1.5k, Resistor_THT:R_Axial_DIN0204_L3.6mm_D1.6mm_P5.08mm_Horizontal, symbol Device:R_US
- added R_Gate-Protect_Boost: 100, Resistor_THT:R_Axial_DIN0204_L3.6mm_D1.6mm_P5.08mm_Horizontal, symbol Device:R_US
- added R_Pull-Down_Boost: 100k, Resistor_THT:R_Axial_DIN0204_L3.6mm_D1.6mm_P5.08mm_Horizontal, symbol Device:R_US
- added U4: NE555P, digikey-footprints:DIP-8_W7.62mm, symbol dk_Clock-Timing-Programmable-Timers-and-Oscillators:NE555P
- SW3: value DIR+A -> PWM_A; footprint (none) -> Button_Switch_THT:SW_PUSH_6mm_H5mm
- SW4: value DIR-A -> DIR_A; footprint (none) -> Button_Switch_THT:SW_PUSH_6mm_H5mm
Connections:
- net +5V: now also J3.7 (Pin_7)
- net GND: now also C10.2, C9.2, R9.1, R_Pull-Down_Boost.1, U4.1 (GND)
- net GND2: now also J3.1 (Pin_1), J3.6 (Pin_6), Q9.2 (S), R10.1; no longer U2.2 (C1), U2.8 (C4)
- net ML-A: now also D10.1 (K), D7.2 (A)
- net MR-A: now also D8.1 (K), D9.2 (A)
- net V_Gate-Boost: now also R_Gate-Protect_Boost.2, R_Pull-Down_Boost.2
- net V_LS-A: now also R11.2, U4.4 (RESET), U4.8 (VCC)
- net Vcc: now also D11.2 (A)
- net GSig_Q1A renamed LED_An_+_A
- net LED_An_+_A: now also J3.3 (Pin_3), Q8.2 (S)
- net GSig_Q2A renamed LED_An_-_A
- net LED_An_-_A: now also Q8.3 (D); no longer SW4.2 (B)
- new net: D10.2 (A), R8.1
- new net: D9.1 (K), R8.2
- new net: R11.1, R12.2, U4.7 (DISCH)
- new net: R_Gate-Protect_Boost.1, U4.3 (OUT)
- new net: C10.1, R12.1, U4.2 (TRIG), U4.6 (THRES)
- new net: C9.1, U4.5 (CONT)
- new net: D7.1 (K), R7.2
- new net: D12.2 (A), Q8.1 (G)
- new net: D8.2 (A), R7.1
- new net: D11.1 (K), R9.2
- new net DIR_A: D12.1 (K), J3.2 (Pin_2), Q9.1 (G), R10.2, SW4.2 (B)
- new net DIR_B: J3.5 (Pin_5)
- new net LED_Ct_+_A: Q9.3 (D), U2.2 (C1), U2.8 (C4)
- new net PWM_B: J3.4 (Pin_4)
Other:
- note added: "Output filter capacitors"
- note removed: "!! Idiot Proof the H-Bridge !!"
- note removed: "H-Bridge Ch-B"
- note removed: "Output filter capacitors indication leds On indication LEDs"
- note removed: "add 2 resistors"
- moved on the sheet: 5V-J1, 5V-J2, C4, C5, C6, C7, C8, D6, F1, J1, J4, L2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

Commit message: Added NMOS Gate Drivers
Parts:
- removed 12V-J1, 12V-J2, 5V-J1: J-12V, Connector_PinHeader_2.54mm:PinHeader_1x02_P2.54mm_Vertical, symbol Jumper:Jumper_2_Open
- removed C2: 100nF, Capacitor_THT:C_Disc_D9.0mm_W5.0mm_P5.00mm, symbol Device:C
- removed C3: 1uF, Capacitor_THT:C_Disc_D9.0mm_W5.0mm_P5.00mm, symbol Device:C
- removed D2, D4, D5: 1N5352B, Diode_THT:D_DO-41_SOD81_P10.16mm_Horizontal, symbol Device:D_Zener
- removed JP1: 24V-J1, Connector_PinHeader_2.54mm:PinHeader_1x02_P2.54mm_Vertical, symbol Jumper:Jumper_2_Bridged
- removed R4: 3.3k, Resistor_THT:R_Axial_DIN0204_L3.6mm_D1.6mm_P5.08mm_Horizontal, symbol Device:R_US
- removed U1: LM317T, Package_TO_SOT_THT:TO-220F-3_Vertical, symbol dk_PMIC-Voltage-Regulators-Linear:LM317T
- added C_Filter_Left1, C_Filter_Right1: 1000uF, Capacitor_THT:CP_Radial_D18.0mm_P7.50mm, symbol Device:C_Polarized_US
- added D1: 1N5352B, Diode_THT:D_DO-41_SOD81_P10.16mm_Horizontal, symbol Device:D_Zener
- C1: value 10uF -> 100uF
- C2: renamed from C10; value (none) -> 100nF
- R1: value 500 -> 100
- R2: value 10k -> 68k
- R3: value 270 -> 33k
- R4: renamed from R11; value ~ -> 1k
- R5: renamed from R12; value ~ -> 33k
- U2: renamed from U4; footprint digikey-footprints:DIP-8_W7.62mm -> Package_DIP:DIP-8_W7.62mm
- renumbered C9 to C3, D11 to D10, D1 to D2, D12 to D4, D7 to D5, D8 to D6, D6 to D7, D9 to D8, D10 to D9, J4 to J2, Q4 to Q3, Q5 to Q4, Q6 to Q5, Q7 to Q6, Q3 to Q7, R8 to R10, R9 to R11, R10 to R6, R5 to R8, R6 to R9, R_Gate-Protect_Boost to R_Gate-Protect_Boost1, R_Pull-Down_Boost to R_Pull-Down_Boost1, SW3 to SW1, SW4 to SW2, U2 to U1
Connections:
- net +5V: now also C7.1, C8.1, L2.2, R8.2
- net GND: now also D3.2 (A)
- net GPow_Q2A: no longer D3.1 (K)
- net ML-A: now also C_Filter_Left1.1
- net MR-A: now also C_Filter_Right1.1; no longer D3.2 (A)
- net V_HS-A: now also R3.1, D1.2 (A)
- net V_LS-A: now also D3.1 (K)
- net Vcc: now also D1.1 (K)
- net at D9.2 (A), R10.1: now also C_Filter_Right1.2
- net at D6.2 (A), R7.1: now also C_Filter_Left1.2
Other:
- note added: "Possiblity of a switch"
- note removed: "Output filter capacitors"
- moved on the sheet: 5V-J2, C1, C2, C3, C4, C5, C6, C7, C8, D10, D2, D5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
